Commit message: 修改一个urdf,加载飞机和云台模型,使用球关节连接

File: assets/urdf/dof_spherical_joint_test.urdf (robot description, URDF)
Before this commit: robot spherical_joint_robot, 5 links, 4 joints
Links:
- removed link base_link
- removed link object
- added link predator, mass 100; collision mesh filename=package://assets/urdf/uav/meshes/predator_without_sphere.obj scale=2.0 2.0 2.0; visual mesh filename=package://assets/urdf/uav/meshes/predator_without_sphere.obj scale=2.0 2.0 2.0
- added link sphere, mass 5; collision mesh filename=package://assets/urdf/uav/meshes/sphere.obj scale=2.0 2.0 2.0; visual mesh filename=package://assets/urdf/uav/meshes/sphere.obj scale=2.0 2.0 2.0
Joints:
- joint prismatic_joint_x: limit lower=-2 upper=2 effort=1000.0 velocity=100 -> lower=-2 upper=2 effort=1.0 velocity=0.1; origin xyz=0 0 0 -> xyz=2.17672 0 -0.119422; parent base_link -> predator
- joint prismatic_joint_y: limit lower=-2 upper=2 effort=1000.0 velocity=100 -> lower=-2 upper=2 effort=1.0 velocity=0.1
- joint prismatic_joint_z: limit lower=-2 upper=2 effort=1000.0 velocity=100 -> lower=-2 upper=2 effort=1.0 velocity=0.1
- joint spherical_joint: child object -> sphere
